File: schematic/eagle/digital-psu.sch (EAGLE design)
At the start: 79 parts, among them IC1 TL072P, IC2 TLC272P, Q1 MPSA56-TO92, T3 2N3055, T4 2N3055, T5 2N3055, X1 Vout, X2 PASS_TRANSISTORS, X3 AC_IN

Commit message: removed all airwires
Connections:
- removed net N$32: C14.2, IC2B.-IN, R25.1, R26/1.A, R26/2.A
- net ADJ_VOLT: now also R25.1, R26/1.A, R26/2.A; no longer R26/1.S, R26/2.S
- net GND_HIGHER: now also C14.2
- net N$2: now also IC2B.-IN, R26/1.S, R26/2.S; no longer R12/1.E, R12/2.E, R13.1
- net N$20: now also R12/1.E, R12/2.E, R13.1
