File: schematic/digital-psu.brd (EAGLE design)
At the start: 100 x 80 mm, 78 parts, among them IC1 TL072P, IC2 TLC272P, Q1 MPSA56-TO92, T1 2N3704, T2 2N3704, T3 2N3055, T4 2N3055, T5 2N3055, T6 2N3704, X1 Vout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

Commit message: created gerber files
Parts:
- removed T6: 2N3704, transistor:TO92
- added T7: (no value), transistor:TO92-EBC
- added VCC: VNEG, con-wago-500:W237-103
- C1, C2, C3: device resistor:EB35D -> resistor:EB22,5D
- R27: value 0k -> 10k; device eagle-ltspice:R0805 -> rcl:RTRIM64W
- T1, T2: value 2N3704 -> (none); device transistor:TO92 -> transistor:TO92-EBC
- moved T5 248.3 mm to (132.1, 20.3)
- moved R18 244.1 mm to (115.6, 59.7)
- moved R17 231.8 mm to (115.6, 34.3)
- moved R16 223.8 mm to (115.6, 7.62)
- moved X1 209.0 mm to (95.2, 29.2), turned to 90 degrees
- moved T4 205.7 mm to (130.8, 73.7)
- moved R30 204.2 mm to (72.4, 52.1), flipped to the bottom
- moved C11 203.5 mm to (61.0, 41.9), flipped to the bottom, turned to 270 degrees
- moved C15 202.6 mm to (55.9, 47.0), flipped to the bottom, turned to 180 degrees
- moved R29 198.6 mm to (73.7, 55.9), flipped to the bottom, turned to 90 degrees
- moved C3 197.1 mm to (91.4, 8.89), turned to 270 degrees
- moved R2 195.8 mm to (57.1, 16.5), flipped to the bottom, turned to 270 degrees
- moved R21 195.5 mm to (97.8, 61.0), flipped to the bottom, turned to 270 degrees
- moved R1 191.6 mm to (33.0, 24.1), flipped to the bottom, turned to 270 degrees
- moved T2 191.6 mm to (63.5, 33.0), turned to 180 degrees
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Connections:
- removed net N$10 (its old number): R29.1, R30.1, T6.1
- removed net N$18 (its old number): D10.A, IC2.3
- removed net N$21: C10.1, C9.1, C9.2, IC2.1, IC2.2, R14.2, R15.1, R20.2, T6.2
- removed net N$22 (its old number): R25.1, R26.1-1, R26.2-1
- removed net N$35 (its old number): R26.1-3, R26.2-3, R27.1
- new net ADJ_VOLT: D10.A, IC2.3, R25.1, R26.1-1, R26.2-1
- new net N$17: R29.1, R30.1, T1.B
- new net N$36: R26.1-3, R26.2-3, R27.1, R27.2
- new net N$38: C10.1, C9.1, IC2.2, R14.2, R20.2
- new net N$41: C10.2, C12.+, D11.A, D12.C, R19.1, R20.1, R21.1, X1.2, X2.1
- new net N$9: T5.C
- net GND: now also T1.E, VCC.2; no longer T6.3
- net GND_HIGHER: now also R27.3; no longer R27.2
- net N$1: now also X3.2; no longer X3.4
- net N$16: now also T7.B; no longer T1.1
- net N$19: now also T7.E; no longer T1.3
- net N$27: now also T2.E; no longer T2.3
- net N$28: now also T2.B; no longer T2.1
- net N$3: now also X3.4; no longer X3.2
- net N$31: now also C9.2, IC2.1, R15.1, T1.C; no longer C10.2, C12.+, D11.A, D12.C, R16.2, R17.2, R18.2, R19.1, R20.1, R21.1, X1.2, X2.1
- net VCC: now also T2.C, T7.C, VCC.1; no longer T1.2, T2.2, T3.C, T4.C, T5.C
- net VNEG: now also VCC.3
Routing:
- net VCC: track 0.00 -> 362.5 mm, vias 0 -> 5
- net VNEG: track 0.00 -> 272.2 mm, vias 0 -> 8
- net GND_HIGHER: track 0.00 -> 173.1 mm, vias 0 -> 3
- net N$41: track 0.00 -> 124.4 mm, vias 0 -> 2
- net N$4: track 0.00 -> 114.2 mm, vias 0 -> 4
- net N$2: track 0.00 -> 95.9 mm, vias 0 -> 2
- net N$30: track 0.00 -> 83.5 mm, vias 0 -> 2
- net N$20: track 0.00 -> 82.1 mm
- net ADJ_VOLT: track 0.00 -> 79.8 mm, vias 0 -> 2
- net ADJ_CURR: track 0.00 -> 56.8 mm, vias 0 -> 4
- net N$38: track 0.00 -> 50.4 mm, vias 0 -> 2
- net N$36: track 0.00 -> 45.1 mm
- net VZENER: track 0.00 -> 44.6 mm, vias 0 -> 2
- net N$28: track 0.00 -> 42.8 mm, vias 0 -> 2
- net N$34: track 0.00 -> 39.7 mm, vias 0 -> 2
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- added copper zone on layer 16, net GND
- added copper zone on layer 1, net N$13
Other:
- board size 100 x 80 mm -> 107.6 x 85.1 mm
- board text added: "DLR PSU"

Commit message: added spice: dac, negative transformer, zener etc, and initial arduino uno code
Connections:
- new net N$32: R12.1-3, R12.2-3, R13.1
- net ADJ_VOLT: now also R26.1-2, R26.2-2; no longer R25.1, R26.1-1, R26.2-1
- net N$2: now also R25.1, R26.1-1, R26.2-1; no longer R26.1-2, R26.2-2
- net N$20: no longer R12.1-3, R12.2-3, R13.1
Routing:
- net N$36: track 45.1 -> 51.8 mm
- net ADJ_VOLT: track 79.8 -> 82.3 mm
Changed lines of the file:
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@@
 <contactref element="R11" pad="1"/>
 <contactref element="C13" pad="2"/>
-<contactref element="R12" pad="1-3"/>
-<contactref element="R12" pad="2-3"/>
-<contactref element="R13" pad="1"/>
 <contactref element="IC1" pad="6"/>
 <wire x1="53.34" y1="66.04" x2="53.34" y2="77.47" width="1.27" layer="16"/>
@@
 <wire x1="2.54" y1="72.39" x2="2.54" y2="62.23" width="1.27" layer="16"/>
 <wire x1="2.54" y1="62.23" x2="10.16" y2="62.23" width="1.27" layer="16"/>
-<wire x1="53.02" y1="72.39" x2="53.02" y2="74.93" width="0" layer="19" extent="16-16"/>
 <wire x1="53.02" y1="69.85" x2="53.02" y2="72.39" width="0" layer="19" extent="16-16"/>
-<wire x1="53.34" y1="77.47" x2="53.02" y2="74.93" width="0" layer="19" extent="16-16"/>
+<wire x1="53.34" y1="66.04" x2="53.02" y2="69.85" width="0" layer="19" extent="16-16"/>
 <wire x1="10.08" y1="72.31" x2="10.16" y2="72.39" width="0" layer="19" extent="16-16"/>
-<wire x1="10.08" y1="62.31" x2="10.16" y2="62.23" width="0" layer="19" extent="16-16"/>
 <wire x1="5.08" y1="72.31" x2="2.54" y2="72.39" width="0" layer="19" extent="16-16"/>
-<wire x1="5.08" y1="62.31" x2="2.54" y2="62.23" width="0" layer="19" extent="16-16"/>
 </signal>
 <signal name="N$23">
@@
 <contactref element="X2" pad="2"/>
 <contactref element="T2" pad="E"/>
+<wire x1="130.302" y1="52.451" x2="129.032" y2="79.121" width="0" layer="19" extent="1-1"/>
 <wire x1="130.302" y1="25.781" x2="130.302" y2="52.451" width="0" layer="19" extent="1-1"/>
-<wire x1="129.032" y1="79.121" x2="130.302" y2="52.451" width="0" layer="19" extent="1-1"/>
 <wire x1="96.54" y1="44.45" x2="130.302" y2="52.451" width="0" layer="19" extent="1-1"/>
 <wire x1="95.57" y1="64.77" x2="96.54" y2="44.45" width="0" layer="19" extent="16-16"/>
@@
 </signal>
 <signal name="ADJ_VOLT">
-<contactref element="R25" pad="1"/>
-<contactref element="R26" pad="2-1"/>
-<contactref element="R26" pad="1-1"/>
 <contactref element="D10" pad="A"/>
 <contactref element="IC2" pad="3"/>
@@
 <wire x1="18.415" y1="46.355" x2="18.415" y2="53.975" width="1.016" layer="1"/>
 <via x="18.415" y="53.975" extent="1-16" drill="0.6" shape="square"/>
-<wire x1="18.415" y1="53.975" x2="10.16" y2="53.975" width="1.016" layer="16"/>
-<wire x1="10.08" y1="54.53" x2="11.75" y2="57.15" width="0" layer="19" extent="16-16"/>
-<wire x1="10.16" y1="53.975" x2="10.08" y2="54.53" width="0" layer="19" extent="16-16"/>
-<wire x1="5.08" y1="54.53" x2="10.08" y2="54.53" width="0" layer="19" extent="1-1"/>
+<wire x1="18.415" y1="53.975" x2="12.7" y2="53.975" width="1.016" layer="16"/>
+<contactref element="R26" pad="2-2"/>
+<contactref element="R26" pad="1-2"/>
+<wire x1="5.08" y1="49.53" x2="10.08" y2="49.53" width="1.27" layer="16"/>
+<wire x1="10.08" y1="49.53" x2="12.7" y2="53.975" width="0" layer="19" extent="16-16"/>
 </signal>
 <signal name="N$2">
-<contactref element="R26" pad="1-2"/>
-<contactref element="R26" pad="2-2"/>
 <contactref element="IC2" pad="6"/>
 <wire x1="71.12" y1="71.755" x2="44.45" y2="71.755" width="1.016" layer="1"/>
@@
 <wire x1="13.97" y1="66.04" x2="13.97" y2="52.07" width="1.016" layer="1"/>
 <via x="13.97" y="52.07" extent="1-16" drill="0.6" shape="square"/>
-<wire x1="5.08" y1="49.53" x2="13.97" y2="49.53" width="1.016" layer="16"/>
 <wire x1="13.97" y1="49.53" x2="13.97" y2="52.07" width="1.016" layer="16"/>
 <wire x1="68.58" y1="62.23" x2="71.12" y2="64.77" width="1.016" layer="16"/>
 <wire x1="71.12" y1="64.77" x2="71.12" y2="71.755" width="1.016" layer="16"/>
 <via x="71.12" y="71.755" extent="1-16" drill="0.6" shape="square"/>
-<wire x1="13.97" y1="49.53" x2="10.08" y2="49.53" width="0" layer="19" extent="16-16"/>
+<contactref element="R25" pad="1"/>
+<contactref element="R26" pad="2-1"/>
+<contactref element="R26" pad="1-1"/>
+<wire x1="5.08" y1="54.53" x2="10.08" y2="54.53" width="1.27" layer="16"/>
+<wire x1="10.08" y1="54.53" x2="10.16" y2="54.53" width="1.27" layer="16"/>
+<wire x1="10.16" y1="54.53" x2="10.16" y2="54.61" width="1.27" layer="16"/>
+<wire x1="11.75" y1="57.15" x2="11.43" y2="57.15" width="1.27" layer="16"/>
+<wire x1="11.43" y1="57.15" x2="10.16" y2="55.88" width="1.27" layer="16"/>
+<wire x1="10.16" y1="55.88" x2="10.16" y2="54.61" width="1.27" layer="16"/>
+<wire x1="10.16" y1="54.61" x2="13.97" y2="54.61" width="0" layer="19" extent="1-16"/>
 </signal>
 <signal name="N$4">
@@
 <wire x1="43.815" y1="40.64" x2="13.97" y2="40.64" width="1.27" layer="16"/>
 <wire x1="13.97" y1="40.64" x2="13.97" y2="44.45" width="1.27" layer="16"/>
-<wire x1="13.97" y1="44.45" x2="5.08" y2="44.45" width="1.27" layer="16"/>
 <wire x1="43.815" y1="40.64" x2="43.815" y2="38.1" width="1.27" layer="16"/>
-<wire x1="13.97" y1="44.45" x2="10.08" y2="44.53" width="0" layer="19" extent="16-16"/>
-<wire x1="5.08" y1="44.53" x2="5.08" y2="44.45" width="0" layer="19" extent="16-16"/>
+<wire x1="5.08" y1="44.45" x2="13.97" y2="44.45" width="1.27" layer="16"/>
+<wire x1="12.7" y1="44.45" x2="10.08" y2="44.45" width="1.27" layer="16"/>
+<wire x1="10.08" y1="44.45" x2="10.08" y2="44.53" width="1.27" layer="16"/>
+<wire x1="10.08" y1="44.53" x2="13.97" y2="44.53" width="1.27" layer="16"/>
+<wire x1="13.97" y1="44.53" x2="13.97" y2="44.45" width="1.27" layer="16"/>
+<wire x1="5.08" y1="44.45" x2="5.08" y2="44.53" width="0" layer="19" extent="16-16"/>
 </signal>
 <signal name="N$35">
@@
 </polygon>
 </signal>
+<signal name="N$32">
+<contactref element="R12" pad="1-3"/>
+<contactref element="R12" pad="2-3"/>
+<contactref element="R13" pad="1"/>
+<wire x1="10.08" y1="62.31" x2="53.02" y2="74.93" width="0" layer="19" extent="16-16"/>
+<wire x1="5.08" y1="62.31" x2="10.08" y2="62.31" width="0" layer="19" extent="1-1"/>
+</signal>
 </signals>
