File: schematic/digital-psu.sch (EAGLE design)
At the start: 78 parts, among them IC1 TL072P, IC2 TLC272P, Q1 MPSA56-TO92, T1 2N3704, T2 2N3704, T3 2N3055, T4 2N3055, T5 2N3055, T6 2N3704, X1 Vout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

Commit message: created gerber files
Parts:
- removed T6: 2N3704, transistor:2N3704
- added T7: (no value), transistor:-NPN-TO92-EBC
- added VCC: VNEG, con-wago-500:W237-103
- C1, C2, C3: device resistor:CPOL-EUE10-35 -> resistor:CPOL-EUE10-22.5
- R27: value 0k -> 10k; device eagle-ltspice:R -> rcl:R-TRIMM64W
- T1, T2: value 2N3704 -> (none); device transistor:2N3704 -> transistor:-NPN-TO92-EBC
Connections:
- removed net N$10 (its old number): R29.1, R30.1, T6.B
- removed net N$18 (its old number): D10.A, IC2A.+IN
- removed net N$21: C10.1, C9.1, C9.2, IC2A.-IN, IC2A.OUT, R14.2, R15.1, R20.2, T6.C
- removed net N$22 (its old number): R25.1, R26/1.A, R26/2.A
- removed net N$35 (its old number): R26/1.E, R26/2.E, R27.1
- new net ADJ_VOLT: D10.A, IC2A.+IN, R25.1, R26/1.A, R26/2.A
- new net N$17: R29.1, R30.1, T1.B
- new net N$36: R26/1.E, R26/2.E, R27.A, R27.S
- new net N$38: C10.1, C9.1, IC2A.-IN, R14.2, R20.2
- new net N$41: C10.2, C12.+, D11.A, D12.C, R19.1, R20.1, R21.1, X1-2.KL, X2-1.KL
- new net N$9: T5.C
- net GND: now also T1.E, VCC-2.KL; no longer T6.E
- net GND_HIGHER: now also R27.E; no longer R27.2
- net N$1: now also X3-2.KL; no longer X3-4.KL
- net N$16: now also T7.B; no longer T1.B
- net N$19: now also T7.E; no longer T1.E
- net N$3: now also X3-4.KL; no longer X3-2.KL
- net N$31: now also C9.2, IC2A.OUT, R15.1, T1.C; no longer C10.2, C12.+, D11.A, D12.C, R16.2, R17.2, R18.2, R19.1, R20.1, R21.1, X1-2.KL, X2-1.KL
- net VCC: now also T7.C, VCC-1.KL; no longer T1.C, T3.C, T4.C, T5.C
- net VNEG: now also VCC-3.KL
Other:
- moved on the sheet: C10, R14, R20, T1

Commit message: added spice: dac, negative transformer, zener etc, and initial arduino uno code
Connections:
- new net N$32: R12/1.E, R12/2.E, R13.1
- net ADJ_VOLT: now also R26/1.S, R26/2.S; no longer R25.1, R26/1.A, R26/2.A
- net N$2: now also R25.1, R26/1.A, R26/2.A; no longer R26/1.S, R26/2.S
- net N$20: no longer R12/1.E, R12/2.E, R13.1
Other:
- moved on the sheet: R26/1, R26/2
Changed lines of the file:
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@@
 <instance part="R17" gate="G$1" x="325.12" y="309.88"/>
 <instance part="R18" gate="G$1" x="320.04" y="299.72"/>
-<instance part="R26" gate="/1" x="320.04" y="208.28" rot="R180"/>
-<instance part="R26" gate="/2" x="304.8" y="208.28" rot="R180"/>
+<instance part="R26" gate="/1" x="320.04" y="208.28" rot="MR180"/>
+<instance part="R26" gate="/2" x="304.8" y="208.28" rot="MR180"/>
 <instance part="S1" gate="1" x="157.48" y="190.5" rot="MR0"/>
 <instance part="S2" gate="1" x="246.38" y="213.36" rot="R90"/>
@@
 <pinref part="R11" gate="G$1" pin="1"/>
 <wire x1="172.72" y1="241.3" x2="190.5" y2="241.3" width="0.1524" layer="91"/>
-<wire x1="190.5" y1="243.84" x2="190.5" y2="254" width="0.1524" layer="91"/>
+<wire x1="190.5" y1="241.3" x2="190.5" y2="254" width="0.1524" layer="91"/>
 <wire x1="190.5" y1="254" x2="185.42" y2="254" width="0.1524" layer="91"/>
 <pinref part="C13" gate="G$1" pin="2"/>
@@
 <junction x="198.12" y="254"/>
 <junction x="190.5" y="254"/>
-<wire x1="190.5" y1="241.3" x2="190.5" y2="243.84" width="0.1524" layer="91"/>
-<pinref part="R12" gate="/1" pin="E"/>
-<pinref part="R12" gate="/2" pin="E"/>
-<wire x1="213.36" y1="243.84" x2="198.12" y2="243.84" width="0.1524" layer="91"/>
-<pinref part="R13" gate="G$1" pin="1"/>
-<wire x1="198.12" y1="241.3" x2="198.12" y2="243.84" width="0.1524" layer="91"/>
-<junction x="198.12" y="243.84"/>
-<wire x1="190.5" y1="243.84" x2="198.12" y2="243.84" width="0.1524" layer="91"/>
-<junction x="190.5" y="243.84"/>
 <pinref part="IC1" gate="B" pin="-IN"/>
 <wire x1="154.94" y1="251.46" x2="154.94" y2="241.3" width="0.1524" layer="91"/>
-<wire x1="154.94" y1="241.3" x2="170.18" y2="241.3" width="0.1524" layer="91"/>
-<wire x1="170.18" y1="241.3" x2="172.72" y2="241.3" width="0.1524" layer="91"/>
+<wire x1="154.94" y1="241.3" x2="172.72" y2="241.3" width="0.1524" layer="91"/>
 <junction x="172.72" y="241.3"/>
 </segment>
@@
 <net name="ADJ_VOLT" class="0">
 <segment>
-<pinref part="R25" gate="G$1" pin="1"/>
-<pinref part="R26" gate="/2" pin="A"/>
-<wire x1="292.1" y1="213.36" x2="304.8" y2="213.36" width="0.1524" layer="91"/>
-<pinref part="R26" gate="/1" pin="A"/>
-<wire x1="304.8" y1="213.36" x2="320.04" y2="213.36" width="0.1524" layer="91"/>
-<junction x="304.8" y="213.36"/>
-<label x="312.42" y="215.9" size="1.778" layer="95" rot="R180"/>
-</segment>
-<segment>
 <wire x1="256.54" y1="287.02" x2="254" y2="287.02" width="0.1524" layer="91"/>
 <wire x1="254" y1="287.02" x2="254" y2="307.34" width="0.1524" layer="91"/>
@@
 <label x="259.08" y="309.88" size="1.778" layer="95" rot="R180"/>
 </segment>
+<segment>
+<pinref part="R26" gate="/2" pin="S"/>
+<pinref part="R26" gate="/1" pin="S"/>
+<wire x1="309.88" y1="208.28" x2="325.12" y2="208.28" width="0.1524" layer="91"/>
+<wire x1="325.12" y1="208.28" x2="330.2" y2="208.28" width="0.1524" layer="91"/>
+<junction x="325.12" y="208.28"/>
+</segment>
 </net>
 <net name="N$2" class="0">
 <segment>
-<pinref part="R26" gate="/1" pin="S"/>
-<pinref part="R26" gate="/2" pin="S"/>
-<wire x1="314.96" y1="208.28" x2="299.72" y2="208.28" width="0.1524" layer="91"/>
-<wire x1="299.72" y1="208.28" x2="287.02" y2="208.28" width="0.1524" layer="91"/>
-<junction x="299.72" y="208.28"/>
-<wire x1="287.02" y1="208.28" x2="287.02" y2="203.2" width="0.1524" layer="91"/>
 <pinref part="IC2" gate="B" pin="-IN"/>
 <wire x1="261.62" y1="210.82" x2="259.08" y2="210.82" width="0.1524" layer="91"/>
-<wire x1="259.08" y1="210.82" x2="259.08" y2="203.2" width="0.1524" layer="91"/>
-<wire x1="287.02" y1="203.2" x2="259.08" y2="203.2" width="0.1524" layer="91"/>
+<wire x1="259.08" y1="210.82" x2="259.08" y2="205.74" width="0.1524" layer="91"/>
+<wire x1="259.08" y1="205.74" x2="297.18" y2="205.74" width="0.1524" layer="91"/>
+<pinref part="R25" gate="G$1" pin="1"/>
+<pinref part="R26" gate="/2" pin="A"/>
+<wire x1="292.1" y1="213.36" x2="297.18" y2="213.36" width="0.1524" layer="91"/>
+<pinref part="R26" gate="/1" pin="A"/>
+<wire x1="297.18" y1="213.36" x2="304.8" y2="213.36" width="0.1524" layer="91"/>
+<wire x1="304.8" y1="213.36" x2="320.04" y2="213.36" width="0.1524" layer="91"/>
+<junction x="304.8" y="213.36"/>
+<label x="312.42" y="215.9" size="1.778" layer="95" rot="R180"/>
+<wire x1="297.18" y1="205.74" x2="297.18" y2="213.36" width="0.1524" layer="91"/>
+<junction x="297.18" y="213.36"/>
 </segment>
 </net>
@@
 </segment>
 </net>
+<net name="N$32" class="0">
+<segment>
+<pinref part="R12" gate="/1" pin="E"/>
+<pinref part="R12" gate="/2" pin="E"/>
+<wire x1="213.36" y1="243.84" x2="198.12" y2="243.84" width="0.1524" layer="91"/>
+<junction x="198.12" y="243.84"/>
+<pinref part="R13" gate="G$1" pin="1"/>
+<wire x1="198.12" y1="241.3" x2="198.12" y2="243.84" width="0.1524" layer="91"/>
+</segment>
+</net>
